Commit message: update

File: src/ia_robot_ros/ia_robot_urdf/urdf/ia_robot.urdf (robot description, URDF)
Before this commit: robot ia_robot, 33 links, 32 joints
Joints:
- joint ARM0_RIGHT: limit lower=-0.04 upper=0.04 effort=100 velocity=1.0 -> lower=0.0 upper=0.04 effort=100 velocity=1.0

File: src/ia_robot_ros/ia_robot_urdf/urdf/ia_robot_ik.absolute.urdf (robot description, URDF)
Before this commit: robot ia_robot, 28 links, 27 joints
Links:
- link ARM0_LEFT: geometry collision mesh filename=package://ia_robot_urdf/meshes/ARM0_LEFT.STL; visual mesh filename=package://ia_robot_urdf/meshes/ARM0_LEFT.STL
- link ARM0_RIGHT: geometry collision mesh filename=package://ia_robot_urdf/meshes/ARM0_RIGHT.STL; visual mesh filename=package://ia_robot_urdf/meshes/ARM0_RIGHT.STL
- link ARM1_LEFT: geometry collision mesh filename=package://ia_robot_urdf/meshes/ARM1_LEFT.STL; visual mesh filename=package://ia_robot_urdf/meshes/ARM1_LEFT.STL
- link ARM1_RIGHT: geometry collision mesh filename=package://ia_robot_urdf/meshes/ARM1_RIGHT.STL; visual mesh filename=package://ia_robot_urdf/meshes/ARM1_RIGHT.STL
- link ARM2_LEFT: geometry collision mesh filename=package://ia_robot_urdf/meshes/ARM2_LEFT.STL; visual mesh filename=package://ia_robot_urdf/meshes/ARM2_LEFT.STL
- link ARM2_RIGHT: geometry collision mesh filename=package://ia_robot_urdf/meshes/ARM2_RIGHT.STL; visual mesh filename=package://ia_robot_urdf/meshes/ARM2_RIGHT.STL
- link ARM3_LEFT: geometry collision mesh filename=package://ia_robot_urdf/meshes/ARM3_LEFT.STL; visual mesh filename=package://ia_robot_urdf/meshes/ARM3_LEFT.STL
- link ARM3_RIGHT: geometry collision mesh filename=package://ia_robot_urdf/meshes/ARM3_RIGHT.STL; visual mesh filename=package://ia_robot_urdf/meshes/ARM3_RIGHT.STL
- link CHEST1: geometry collision mesh filename=package://ia_robot_urdf/meshes/CHEST1.STL; visual mesh filename=package://ia_robot_urdf/meshes/CHEST1.STL
- link Leg_back_left_1: geometry collision mesh filename=package://ia_robot_urdf/meshes/Leg_back_left_1_nocable.STL; visual mesh filename=package://ia_robot_urdf/meshes/Leg_back_left_1_nocable.STL
- link Leg_back_left_2: geometry collision mesh filename=package://ia_robot_urdf/meshes/Leg_back_left_2.STL; visual mesh filename=package://ia_robot_urdf/meshes/Leg_back_left_2.STL
- link Leg_back_right_1: geometry collision mesh filename=package://ia_robot_urdf/meshes/Leg_back_right_1_nocable.STL; visual mesh filename=package://ia_robot_urdf/meshes/Leg_back_right_1_nocable.STL
- link Leg_back_right_2: geometry collision mesh filename=package://ia_robot_urdf/meshes/Leg_back_right_2.STL; visual mesh filename=package://ia_robot_urdf/meshes/Leg_back_right_2.STL
- link Leg_front_left_1: geometry collision mesh filename=package://ia_robot_urdf/meshes/Leg_front_left_1_nocable.STL; visual mesh filename=package://ia_robot_urdf/meshes/Leg_front_left_1_nocable.STL
- link Leg_front_left_2: geometry collision mesh filename=package://ia_robot_urdf/meshes/Leg_front_left_2.STL; visual mesh filename=package://ia_robot_urdf/meshes/Leg_front_left_2.STL
- link Leg_front_left_3: geometry collision mesh filename=package://ia_robot_urdf/meshes/Leg_front_left_3.STL; visual mesh filename=package://ia_robot_urdf/meshes/Leg_front_left_3.STL
- link Leg_front_right_1: geometry collision mesh filename=package://ia_robot_urdf/meshes/Leg_front_right_1_nocable.STL; visual mesh filename=package://ia_robot_urdf/meshes/Leg_front_right_1_nocable.STL
- link Leg_front_right_2: geometry collision mesh filename=package://ia_robot_urdf/meshes/Leg_front_right_2.STL; visual mesh filename=package://ia_robot_urdf/meshes/Leg_front_right_2.STL
- link Leg_front_right_3: geometry collision mesh filename=package://ia_robot_urdf/meshes/Leg_front_right_3.STL; visual mesh filename=package://ia_robot_urdf/meshes/Leg_front_right_3.STL
- link base_link: geometry collision mesh filename=package://ia_robot_urdf/meshes/base_link_col_left.STL; collision mesh filename=package://ia_robot_urdf/meshes/base_link_col_right.STL

File: src/ia_robot_ros/ia_robot_urdf/urdf/ia_robot_model.urdf (robot description, URDF)
Before this commit: robot ia_robot, 33 links, 32 joints
Joints:
- joint ARM0_LEFT: limit lower=-0.04 upper=0.04 effort=100 velocity=1.0 -> lower=0.0 upper=0.04 effort=100 velocity=1.0
- joint ARM0_RIGHT: limit lower=-0.04 upper=0.04 effort=100 velocity=1.0 -> lower=0.0 upper=0.04 effort=100 velocity=1.0
